File: USB 2.0 Hub.kicad_pcb (KiCad board)
At the start: 2 copper layers, 86.5 x 37.5 mm, 36 parts, among them J1 USB_C_Receptacle_USB2.0_16P, J2 USB_A, J3 USB_A, J4 USB_A, J5 USB_A, U1 SRV05-4, U2 SRV05-4, U3 FE1.1s, U4 SRV05-4, Y1 12MHz

Commit message: Added finishing touches to final design and generated BoM
Parts:
- added C8: 100nF, Capacitor_SMD:C_0805_2012Metric_Pad1.18x1.45mm_HandSolder, F.Cu at (171.0, 102.5)
- moved R10 2.45 mm to (168.5, 102.5)
- moved R9 1.95 mm to (165.5, 101.5)
- moved Y1 0.48 mm to (183.9, 97.0)
- moved C5 0.05 mm to (173.5, 102.5)
Routing:
- net +5V: track 203.1 -> 199.1 mm
- net GND: track 35.9 -> 38.2 mm
- net /VBUSM: track 6.75 -> 7.69 mm
- net /OVCJ: track 8.08 -> 7.54 mm
