File: downstream_ports.kicad_sch (KiCad schematic)
At the start: 10 parts, among them J2 USB_A, J3 USB_A, J4 USB_A, J5 USB_A, U1 SRV05-4, U4 SRV05-4

Commit message: Added finishing touches to final design and generated BoM
Parts:
- C1, C3, C6, C7: value 0.1uF -> 100nF
Connections:
- net D3+ is gone; now on net +5V: J4.3 (D+), U4.6 (IO4)
- net D3- is gone; now on net +5V: J4.2 (D-), U4.4 (IO3)
Other:
- moved on the sheet: C1, C3, C6, C7, U1, U4
