File: upstream_port.kicad_sch (KiCad schematic)
At the start: 4 parts, among them J1 USB_C_Receptacle_USB2.0_16P, U2 SRV05-4

Commit message: Added finishing touches to final design and generated BoM
Changed lines of the file:
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@@
+	(wire
+		(pts
+			(xy 111.76 68.58) (xy 107.95 68.58)
+		)
+		(stroke
+			(width 0)
+			(type default)
+		)
+	)
 	(wire
 		(pts
@@
 	(wire
 		(pts
-			(xy 107.95 68.58) (xy 111.76 68.58)
-		)
-		(stroke
-			(width 0)
-			(type default)
-		)
-	)
-	(wire
-		(pts
 			(xy 116.84 97.79) (xy 116.84 102.87)
 		)
@@
 		(pts
 			(xy 107.95 81.28) (xy 109.22 81.28)
+		)
+		(stroke
+			(width 0)
+			(type default)
+		)
+	)
+	(wire
+		(pts
+			(xy 111.76 67.31) (xy 111.76 68.58)
 		)
 		(stroke
@@
 	(symbol
 		(lib_id "power:+5V")
-		(at 111.76 68.58 0)
+		(at 111.76 67.31 0)
 		(unit 1)
 		(exclude_from_sim no)
@@
 		(fields_autoplaced yes)
 		(property "Reference" "#PWR06"
-			(at 111.76 72.39 0)
+			(at 111.76 71.12 0)
 			(effects
 				(font
@@
 		)
 		(property "Value" "+5V"
-			(at 111.76 63.5 0)
+			(at 111.76 62.23 0)
 			(effects
 				(font
@@
 		)
 		(property "Footprint" ""
-			(at 111.76 68.58 0)
+			(at 111.76 67.31 0)
 			(effects
 				(font
@@
 		)
 		(property "Datasheet" ""
-			(at 111.76 68.58 0)
+			(at 111.76 67.31 0)
 			(effects
 				(font
@@
 		)
 		(property "Description" "Power symbol creates a global label with name \"+5V\""
-			(at 111.76 68.58 0)
-			(effects
-				(font
+			(at 111.76 67.31 0)
+			(effects
+				(font
